File: hardware/kicad/can_imu.kicad_sch (KiCad schematic)
At the start: 23 parts, among them J3 CAN: H L GND, J4 TERM: shunt=ON, U3 TCAN3413DR, U4 LSM6DSLTR

Commit message: hardware: review schematic and align mechanical and probe attributes
Parts:
- TP10, TP11, TP12, TP7, TP8, TP9: now left out of the parts list
Changed lines of the file:
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@@
 (text "NC10/11 pads soldered; no external reset." (at 233.68 254 0) (effects (font (size 1.27 1.27)) (justify left)))
 (text "Axes: see design_notes.md; verify before PCB." (at 233.68 259.08 0) (effects (font (size 1.27 1.27)) (justify left)))
-(symbol (lib_id "Connector:TestPoint") (at 35.56 228.6 0) (unit 1) (in_bom yes) (on_board yes) (dnp no) (property "Reference" "TP7" (at 40.64 223.51999999999998 0) (effects (font (size 1 1)) (justify left)))(property "Value" "CANH" (at 40.64 226.05999999999997 0) (effects (font (size 1 1)) (justify left)))(property "Footprint" "TestPoint:TestPoint_Pad_D1.5mm" (at 35.56 228.6 0) (effects (font (size 1 1)) (hide yes))) (instances (project "reaction_wheel_controller" (path "/56c7795e-d739-4c45-a73e-6c5ecdfd94b9/abc62b74-3a28-4af7-9f37-2e1e0209501e" (reference "TP7") (unit 1)))))
+(symbol (lib_id "Connector:TestPoint") (at 35.56 228.6 0) (unit 1) (in_bom no) (on_board yes) (dnp no) (property "Reference" "TP7" (at 40.64 223.51999999999998 0) (effects (font (size 1 1)) (justify left)))(property "Value" "CANH" (at 40.64 226.05999999999997 0) (effects (font (size 1 1)) (justify left)))(property "Footprint" "TestPoint:TestPoint_Pad_D1.5mm" (at 35.56 228.6 0) (effects (font (size 1 1)) (hide yes))) (instances (project "reaction_wheel_controller" (path "/56c7795e-d739-4c45-a73e-6c5ecdfd94b9/abc62b74-3a28-4af7-9f37-2e1e0209501e" (reference "TP7") (unit 1)))))
 (wire (pts (xy 35.56 228.6) (xy 35.56 233.68)) (stroke (width 0) (type default)))
 (label "CANH" (at 35.56 233.68 0) (effects (font (size 1 1)) (justify left bottom)))
-(symbol (lib_id "Connector:TestPoint") (at 78.74000000000001 228.6 0) (unit 1) (in_bom yes) (on_board yes) (dnp no) (property "Reference" "TP8" (at 83.82000000000001 223.51999999999998 0) (effects (font (size 1 1)) (justify left)))(property "Value" "CANL" (at 83.82000000000001 226.05999999999997 0) (effects (font (size 1 1)) (justify left)))(property "Footprint" "TestPoint:TestPoint_Pad_D1.5mm" (at 78.74000000000001 228.6 0) (effects (font (size 1 1)) (hide yes))) (instances (project "reaction_wheel_controller" (path "/56c7795e-d739-4c45-a73e-6c5ecdfd94b9/abc62b74-3a28-4af7-9f37-2e1e0209501e" (reference "TP8") (unit 1)))))
+(symbol (lib_id "Connector:TestPoint") (at 78.74000000000001 228.6 0) (unit 1) (in_bom no) (on_board yes) (dnp no) (property "Reference" "TP8" (at 83.82000000000001 223.51999999999998 0) (effects (font (size 1 1)) (justify left)))(property "Value" "CANL" (at 83.82000000000001 226.05999999999997 0) (effects (font (size 1 1)) (justify left)))(property "Footprint" "TestPoint:TestPoint_Pad_D1.5mm" (at 78.74000000000001 228.6 0) (effects (font (size 1 1)) (hide yes))) (instances (project "reaction_wheel_controller" (path "/56c7795e-d739-4c45-a73e-6c5ecdfd94b9/abc62b74-3a28-4af7-9f37-2e1e0209501e" (reference "TP8") (unit 1)))))
 (wire (pts (xy 78.74 228.6) (xy 78.74 233.68)) (stroke (width 0) (type default)))
 (label "CANL" (at 78.74 233.68 0) (effects (font (size 1 1)) (justify left bottom)))
-(symbol (lib_id "Connector:TestPoint") (at 121.92 228.6 0) (unit 1) (in_bom yes) (on_board yes) (dnp no) (property "Reference" "TP9" (at 127.0 223.51999999999998 0) (effects (font (size 1 1)) (justify left)))(property "Value" "FDCAN_TX" (at 127.0 226.05999999999997 0) (effects (font (size 1 1)) (justify left)))(property "Footprint" "TestPoint:TestPoint_Pad_D1.5mm" (at 121.92 228.6 0) (effects (font (size 1 1)) (hide yes))) (instances (project "reaction_wheel_controller" (path "/56c7795e-d739-4c45-a73e-6c5ecdfd94b9/abc62b74-3a28-4af7-9f37-2e1e0209501e" (reference "TP9") (unit 1)))))
+(symbol (lib_id "Connector:TestPoint") (at 121.92 228.6 0) (unit 1) (in_bom no) (on_board yes) (dnp no) (property "Reference" "TP9" (at 127.0 223.51999999999998 0) (effects (font (size 1 1)) (justify left)))(property "Value" "FDCAN_TX" (at 127.0 226.05999999999997 0) (effects (font (size 1 1)) (justify left)))(property "Footprint" "TestPoint:TestPoint_Pad_D1.5mm" (at 121.92 228.6 0) (effects (font (size 1 1)) (hide yes))) (instances (project "reaction_wheel_controller" (path "/56c7795e-d739-4c45-a73e-6c5ecdfd94b9/abc62b74-3a28-4af7-9f37-2e1e0209501e" (reference "TP9") (unit 1)))))
 (wire (pts (xy 121.92 228.6) (xy 121.92 233.68)) (stroke (width 0) (type default)))
 (global_label "FDCAN_TX" (shape bidirectional) (at 121.92 233.68 0) (effects (font (size 1 1)) (justify left bottom)))
-(symbol (lib_id "Connector:TestPoint") (at 165.1 228.6 0) (unit 1) (in_bom yes) (on_board yes) (dnp no) (property "Reference" "TP10" (at 170.18 223.51999999999998 0) (effects (font (size 1 1)) (justify left)))(property "Value" "FDCAN_RX" (at 170.18 226.05999999999997 0) (effects (font (size 1 1)) (justify left)))(property "Footprint" "TestPoint:TestPoint_Pad_D1.5mm" (at 165.1 228.6 0) (effects (font (size 1 1)) (hide yes))) (instances (project "reaction_wheel_controller" (path "/56c7795e-d739-4c45-a73e-6c5ecdfd94b9/abc62b74-3a28-4af7-9f37-2e1e0209501e" (reference "TP10") (unit 1)))))
+(symbol (lib_id "Connector:TestPoint") (at 165.1 228.6 0) (unit 1) (in_bom no) (on_board yes) (dnp no) (property "Reference" "TP10" (at 170.18 223.51999999999998 0) (effects (font (size 1 1)) (justify left)))(property "Value" "FDCAN_RX" (at 170.18 226.05999999999997 0) (effects (font (size 1 1)) (justify left)))(property "Footprint" "TestPoint:TestPoint_Pad_D1.5mm" (at 165.1 228.6 0) (effects (font (size 1 1)) (hide yes))) (instances (project "reaction_wheel_controller" (path "/56c7795e-d739-4c45-a73e-6c5ecdfd94b9/abc62b74-3a28-4af7-9f37-2e1e0209501e" (reference "TP10") (unit 1)))))
 (wire (pts (xy 165.1 228.6) (xy 165.1 233.68)) (stroke (width 0) (type default)))
 (global_label "FDCAN_RX" (shape bidirectional) (at 165.1 233.68 0) (effects (font (size 1 1)) (justify left bottom)))
-(symbol (lib_id "Connector:TestPoint") (at 35.56 259.08 0) (unit 1) (in_bom yes) (on_board yes) (dnp no) (property "Reference" "TP11" (at 40.64 253.99999999999997 0) (effects (font (size 1 1)) (justify left)))(property "Value" "IMU_CS_N" (at 40.64 256.53999999999996 0) (effects (font (size 1 1)) (justify left)))(property "Footprint" "TestPoint:TestPoint_Pad_D1.5mm" (at 35.56 259.08 0) (effects (font (size 1 1)) (hide yes))) (instances (project "reaction_wheel_controller" (path "/56c7795e-d739-4c45-a73e-6c5ecdfd94b9/abc62b74-3a28-4af7-9f37-2e1e0209501e" (reference "TP11") (unit 1)))))
+(symbol (lib_id "Connector:TestPoint") (at 35.56 259.08 0) (unit 1) (in_bom no) (on_board yes) (dnp no) (property "Reference" "TP11" (at 40.64 253.99999999999997 0) (effects (font (size 1 1)) (justify left)))(property "Value" "IMU_CS_N" (at 40.64 256.53999999999996 0) (effects (font (size 1 1)) (justify left)))(property "Footprint" "TestPoint:TestPoint_Pad_D1.5mm" (at 35.56 259.08 0) (effects (font (size 1 1)) (hide yes))) (instances (project "reaction_wheel_controller" (path "/56c7795e-d739-4c45-a73e-6c5ecdfd94b9/abc62b74-3a28-4af7-9f37-2e1e0209501e" (reference "TP11") (unit 1)))))
 (wire (pts (xy 35.56 259.08) (xy 35.56 264.16)) (stroke (width 0) (type default)))
 (global_label "IMU_CS_N" (shape bidirectional) (at 35.56 264.16 0) (effects (font (size 1 1)) (justify left bottom)))
-(symbol (lib_id "Connector:TestPoint") (at 121.92 259.08 0) (unit 1) (in_bom yes) (on_board yes) (dnp no) (property "Reference" "TP12" (at 127.0 253.99999999999997 0) (effects (font (size 1 1)) (justify left)))(property "Value" "IMU_INT1" (at 127.0 256.53999999999996 0) (effects (font (size 1 1)) (justify left)))(property "Footprint" "TestPoint:TestPoint_Pad_D1.5mm" (at 121.92 259.08 0) (effects (font (size 1 1)) (hide yes))) (instances (project "reaction_wheel_controller" (path "/56c7795e-d739-4c45-a73e-6c5ecdfd94b9/abc62b74-3a28-4af7-9f37-2e1e0209501e" (reference "TP12") (unit 1)))))
+(symbol (lib_id "Connector:TestPoint") (at 121.92 259.08 0) (unit 1) (in_bom no) (on_board yes) (dnp no) (property "Reference" "TP12" (at 127.0 253.99999999999997 0) (effects (font (size 1 1)) (justify left)))(property "Value" "IMU_INT1" (at 127.0 256.53999999999996 0) (effects (font (size 1 1)) (justify left)))(property "Footprint" "TestPoint:TestPoint_Pad_D1.5mm" (at 121.92 259.08 0) (effects (font (size 1 1)) (hide yes))) (instances (project "reaction_wheel_controller" (path "/56c7795e-d739-4c45-a73e-6c5ecdfd94b9/abc62b74-3a28-4af7-9f37-2e1e0209501e" (reference "TP12") (unit 1)))))
 (wire (pts (xy 121.92 259.08) (xy 121.92 264.16)) (stroke (width 0) (type default)))
 (global_label "IMU_INT1" (shape bidirectional) (at 121.92 264.16 0) (effects (font (size 1 1)) (justify left bottom)))
