File: hardware/kicad/encoder_esc.kicad_sch (KiCad schematic)
At the start: 25 parts, among them J5 ENC: 3V3 GND A B Z, J6 ESC: PWM EN FAULT GND TX RX, J7 DEBUG: TX RX GND, U5 SN74LVC1G126DBVR

Commit message: hardware: review schematic and align mechanical and probe attributes
Parts:
- TP13, TP14, TP15, TP16: now left out of the parts list
Changed lines of the file:
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@@
 (text "No encoder IC fixed: RPM, PPR, magnet and module still TBD." (at 25.4 198.12 0) (effects (font (size 1.27 1.27)) (justify left)))
 (text "TIM3 A/B, PC3 index. No analog RC filter on edge inputs." (at 25.4 203.2 0) (effects (font (size 1.27 1.27)) (justify left)))
-(symbol (lib_id "Connector:TestPoint") (at 35.56 223.52 0) (unit 1) (in_bom yes) (on_board yes) (dnp no) (property "Reference" "TP13" (at 40.64 218.44 0) (effects (font (size 1 1)) (justify left)))(property "Value" "ENC_A" (at 40.64 220.98 0) (effects (font (size 1 1)) (justify left)))(property "Footprint" "TestPoint:TestPoint_Pad_D1.5mm" (at 35.56 223.52 0) (effects (font (size 1 1)) (hide yes))) (instances (project "reaction_wheel_controller" (path "/56c7795e-d739-4c45-a73e-6c5ecdfd94b9/5febb7f7-899b-4eaf-9fee-36dcc2e6f480" (reference "TP13") (unit 1)))))
+(symbol (lib_id "Connector:TestPoint") (at 35.56 223.52 0) (unit 1) (in_bom no) (on_board yes) (dnp no) (property "Reference" "TP13" (at 40.64 218.44 0) (effects (font (size 1 1)) (justify left)))(property "Value" "ENC_A" (at 40.64 220.98 0) (effects (font (size 1 1)) (justify left)))(property "Footprint" "TestPoint:TestPoint_Pad_D1.5mm" (at 35.56 223.52 0) (effects (font (size 1 1)) (hide yes))) (instances (project "reaction_wheel_controller" (path "/56c7795e-d739-4c45-a73e-6c5ecdfd94b9/5febb7f7-899b-4eaf-9fee-36dcc2e6f480" (reference "TP13") (unit 1)))))
 (wire (pts (xy 35.56 223.52) (xy 35.56 228.6)) (stroke (width 0) (type default)))
 (global_label "ENC_A" (shape bidirectional) (at 35.56 228.6 0) (effects (font (size 1 1)) (justify left bottom)))
-(symbol (lib_id "Connector:TestPoint") (at 121.92 223.52 0) (unit 1) (in_bom yes) (on_board yes) (dnp no) (property "Reference" "TP14" (at 127.0 218.44 0) (effects (font (size 1 1)) (justify left)))(property "Value" "ENC_B" (at 127.0 220.98 0) (effects (font (size 1 1)) (justify left)))(property "Footprint" "TestPoint:TestPoint_Pad_D1.5mm" (at 121.92 223.52 0) (effects (font (size 1 1)) (hide yes))) (instances (project "reaction_wheel_controller" (path "/56c7795e-d739-4c45-a73e-6c5ecdfd94b9/5febb7f7-899b-4eaf-9fee-36dcc2e6f480" (reference "TP14") (unit 1)))))
+(symbol (lib_id "Connector:TestPoint") (at 121.92 223.52 0) (unit 1) (in_bom no) (on_board yes) (dnp no) (property "Reference" "TP14" (at 127.0 218.44 0) (effects (font (size 1 1)) (justify left)))(property "Value" "ENC_B" (at 127.0 220.98 0) (effects (font (size 1 1)) (justify left)))(property "Footprint" "TestPoint:TestPoint_Pad_D1.5mm" (at 121.92 223.52 0) (effects (font (size 1 1)) (hide yes))) (instances (project "reaction_wheel_controller" (path "/56c7795e-d739-4c45-a73e-6c5ecdfd94b9/5febb7f7-899b-4eaf-9fee-36dcc2e6f480" (reference "TP14") (unit 1)))))
 (wire (pts (xy 121.92 223.52) (xy 121.92 228.6)) (stroke (width 0) (type default)))
 (global_label "ENC_B" (shape bidirectional) (at 121.92 228.6 0) (effects (font (size 1 1)) (justify left bottom)))
@@
 (wire (pts (xy 248.92 242.57) (xy 248.92 247.65)) (stroke (width 0) (type default)))
 (global_label "GND" (shape bidirectional) (at 248.92 247.65 0) (effects (font (size 1 1)) (justify left bottom)))
-(symbol (lib_id "Connector:TestPoint") (at 330.2 238.76 0) (unit 1) (in_bom yes) (on_board yes) (dnp no) (property "Reference" "TP15" (at 335.28 233.67999999999998 0) (effects (font (size 1 1)) (justify left)))(property "Value" "ESC_PWM" (at 335.28 236.21999999999997 0) (effects (font (size 1 1)) (justify left)))(property "Footprint" "TestPoint:TestPoint_Pad_D1.5mm" (at 330.2 238.76 0) (effects (font (size 1 1)) (hide yes))) (instances (project "reaction_wheel_controller" (path "/56c7795e-d739-4c45-a73e-6c5ecdfd94b9/5febb7f7-899b-4eaf-9fee-36dcc2e6f480" (reference "TP15") (unit 1)))))
+(symbol (lib_id "Connector:TestPoint") (at 330.2 238.76 0) (unit 1) (in_bom no) (on_board yes) (dnp no) (property "Reference" "TP15" (at 335.28 233.67999999999998 0) (effects (font (size 1 1)) (justify left)))(property "Value" "ESC_PWM" (at 335.28 236.21999999999997 0) (effects (font (size 1 1)) (justify left)))(property "Footprint" "TestPoint:TestPoint_Pad_D1.5mm" (at 330.2 238.76 0) (effects (font (size 1 1)) (hide yes))) (instances (project "reaction_wheel_controller" (path "/56c7795e-d739-4c45-a73e-6c5ecdfd94b9/5febb7f7-899b-4eaf-9fee-36dcc2e6f480" (reference "TP15") (unit 1)))))
 (wire (pts (xy 330.2 238.76) (xy 330.2 243.84)) (stroke (width 0) (type default)))
 (label "ESC_PWM" (at 330.2 243.84 0) (effects (font (size 1 1)) (justify left bottom)))
-(symbol (lib_id "Connector:TestPoint") (at 373.38 238.76 0) (unit 1) (in_bom yes) (on_board yes) (dnp no) (property "Reference" "TP16" (at 378.46 233.67999999999998 0) (effects (font (size 1 1)) (justify left)))(property "Value" "ESC_EN_OUT" (at 378.46 236.21999999999997 0) (effects (font (size 1 1)) (justify left)))(property "Footprint" "TestPoint:TestPoint_Pad_D1.5mm" (at 373.38 238.76 0) (effects (font (size 1 1)) (hide yes))) (instances (project "reaction_wheel_controller" (path "/56c7795e-d739-4c45-a73e-6c5ecdfd94b9/5febb7f7-899b-4eaf-9fee-36dcc2e6f480" (reference "TP16") (unit 1)))))
+(symbol (lib_id "Connector:TestPoint") (at 373.38 238.76 0) (unit 1) (in_bom no) (on_board yes) (dnp no) (property "Reference" "TP16" (at 378.46 233.67999999999998 0) (effects (font (size 1 1)) (justify left)))(property "Value" "ESC_EN_OUT" (at 378.46 236.21999999999997 0) (effects (font (size 1 1)) (justify left)))(property "Footprint" "TestPoint:TestPoint_Pad_D1.5mm" (at 373.38 238.76 0) (effects (font (size 1 1)) (hide yes))) (instances (project "reaction_wheel_controller" (path "/56c7795e-d739-4c45-a73e-6c5ecdfd94b9/5febb7f7-899b-4eaf-9fee-36dcc2e6f480" (reference "TP16") (unit 1)))))
 (wire (pts (xy 373.38 238.76) (xy 373.38 243.84)) (stroke (width 0) (type default)))
 (label "ESC_EN_OUT" (at 373.38 243.84 0) (effects (font (size 1 1)) (justify left bottom)))
